File: Electronics/SmartCup1.brd (EAGLE design)
At the start: 57 x 37 mm, 50 parts, among them IC1 REG1117, IC2 REG1117, SW1 SPST_TACT-EVQQ2

Commit message: Board update
Parts:
- added U$2: TC54VC300, TC54VC27:SOT23
- Q1: device adafruit:SOT223 -> adafruit:SOT23
- moved JP1 118.3 mm to (-61.0, 44.5), turned to 0 degrees
- moved R5 108.2 mm to (-52.1, 52.1), flipped to the top, turned to 0 degrees
- moved R17 106.1 mm to (-69.8, 58.4)
- moved LED4 102.5 mm to (-53.3, 45.7), turned to 0 degrees
- moved C9 100.0 mm to (-43.2, 64.8), turned to 0 degrees
- moved C8 98.6 mm to (-36.8, 64.8), turned to 0 degrees
- moved U$7 98.5 mm to (-54.6, 6.35), flipped to the top
- moved R4 92.3 mm to (-45.7, 52.1), flipped to the top, turned to 0 degrees
- moved R3 90.5 mm to (-39.4, 52.1), flipped to the top, turned to 0 degrees
- moved SW1 88.3 mm to (-57.1, 25.4)
- moved R13 87.5 mm to (-43.2, 58.4), flipped to the top, turned to 0 degrees
- moved R14 82.9 mm to (-49.5, 58.4), flipped to the top, turned to 0 degrees
- moved U$8 80.9 mm to (-66.0, 6.35), flipped to the top
- moved Q1 77.6 mm to (-15.2, 52.1), turned to 0 degrees
- moved R12 76.6 mm to (-36.8, 58.4), flipped to the top, turned to 0 degrees
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Connections:
- new net N$1: Q1.1, U$2.1
- new net N$20: C10.1, C11.1, C12.1, C13.1, C5.1, C6.1, U$1.14, U$1.2, U$1.24, U$1.34, U$1.44, U$1.7
- net LIPO_OUT: now also U$2.3; no longer Q1.1
- net N$8: now also U$2.2
- net VCC: no longer C10.1, C11.1, C12.1, C13.1, C5.1, C6.1, U$1.14, U$1.2, U$1.24, U$1.34, U$1.44, U$1.7
Routing:
- net VCC: track 193.3 -> 0.00 mm
- net LED_R: track 135.1 -> 24.5 mm
- net LIPO_OUT: track 108.2 -> 2.86 mm, vias 2 -> 0
- net LED_G: track 144.8 -> 42.2 mm
- net LED_B: track 126.6 -> 26.2 mm, vias 4 -> 2
- net N$26: track 66.8 -> 0.00 mm, vias 1 -> 0
- net USB_VOUT: track 53.8 -> 23.9 mm
- net N$20: track 0.00 -> 21.2 mm
- net N$8: track 16.5 -> 0.00 mm
- net N$22: track 7.77 -> 0.00 mm
- net N$9: track 7.58 -> 0.00 mm, vias 1 -> 0
- net N$25: track 7.36 -> 0.00 mm
- net N$10: track 7.31 -> 0.00 mm, vias 1 -> 0
- net N$13: track 8.68 -> 1.41 mm, vias 1 -> 0
- net GND: track 45.8 -> 53.0 mm, vias 7 -> 6
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- added copper zone on layer 1, net VCC
- removed copper zone on layer 1, net GND
