File: Electronics/SmartCup.brd (EAGLE design)
At the start: 57 x 37 mm, 50 parts, among them IC1 REG1117, IC2 REG1117, SW1 SPST_TACT-EVQQ2

Commit message: SolidWorks model
Parts:
- R10, R11, R13, R14, R4, R5, R7, R8: value 100m -> 0 Ohm
- R12, R3, R6, R9: value 100m -> 165 Ohm
Changed lines of the file:
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@@
 <element name="C8" library="resistor" package="C0603" value="100nF" x="53.13" y="24.47" rot="R90"/>
 <element name="C9" library="resistor" package="C0603" value="100nF" x="48.37" y="24.58" rot="R270"/>
-<element name="R3" library="resistor" package="R0603" value="100m" x="38.63" y="6.17" rot="MR270"/>
-<element name="R4" library="resistor" package="R0603" value="100m" x="31.57" y="1.68" rot="MR90"/>
-<element name="R5" library="resistor" package="R0603" value="100m" x="44.17" y="2.73" rot="MR90"/>
+<element name="R3" library="resistor" package="R0603" value="165 Ohm" x="38.63" y="6.17" rot="MR270"/>
+<element name="R4" library="resistor" package="R0603" value="0 Ohm" x="31.57" y="1.68" rot="MR90"/>
+<element name="R5" library="resistor" package="R0603" value="0 Ohm" x="44.17" y="2.73" rot="MR90"/>
 <element name="LED1" library="led" package="GM1WA55311A" value="GM1WA55311A" x="18.21" y="35.18" rot="R90"/>
-<element name="R6" library="resistor" package="R0603" value="100m" x="14.63" y="35.045" rot="MR270"/>
-<element name="R7" library="resistor" package="R0603" value="100m" x="19.87" y="31.73" rot="MR90"/>
-<element name="R8" library="resistor" package="R0603" value="100m" x="17.18" y="31.23" rot="MR180"/>
+<element name="R6" library="resistor" package="R0603" value="165 Ohm" x="14.63" y="35.045" rot="MR270"/>
+<element name="R7" library="resistor" package="R0603" value="0 Ohm" x="19.87" y="31.73" rot="MR90"/>
+<element name="R8" library="resistor" package="R0603" value="0 Ohm" x="17.18" y="31.23" rot="MR180"/>
 <element name="LED2" library="led" package="GM1WA55311A" value="GM1WA55311A" x="38.72" y="35.2" rot="R270"/>
-<element name="R9" library="resistor" package="R0603" value="100m" x="30.17" y="35.68" rot="MR180"/>
-<element name="R10" library="resistor" package="R0603" value="100m" x="38.92" y="31.67" rot="MR90"/>
-<element name="R11" library="resistor" package="R0603" value="100m" x="41.12" y="31.72" rot="MR90"/>
+<element name="R9" library="resistor" package="R0603" value="165 Ohm" x="30.17" y="35.68" rot="MR180"/>
+<element name="R10" library="resistor" package="R0603" value="0 Ohm" x="38.92" y="31.67" rot="MR90"/>
+<element name="R11" library="resistor" package="R0603" value="0 Ohm" x="41.12" y="31.72" rot="MR90"/>
 <element name="C10" library="resistor" package="C0603" value="100nF" x="22.63" y="29.98" rot="R180"/>
 <element name="C11" library="resistor" package="C0603" value="100nF" x="34.13" y="30.52" rot="R90"/>
 <element name="C12" library="resistor" package="C0603" value="100nF" x="39.47" y="15.47"/>
 <element name="LED3" library="led" package="GM1WA55311A" value="GM1WA55311A" x="17.18" y="2.13" rot="R90"/>
-<element name="R12" library="resistor" package="R0603" value="100m" x="19.18" y="6.13" rot="MR270"/>
-<element name="R13" library="resistor" package="R0603" value="100m" x="23.43" y="1.68" rot="MR270"/>
-<element name="R14" library="resistor" package="R0603" value="100m" x="14.78" y="6.13" rot="MR270"/>
+<element name="R12" library="resistor" package="R0603" value="165 Ohm" x="19.18" y="6.13" rot="MR270"/>
+<element name="R13" library="resistor" package="R0603" value="0 Ohm" x="23.43" y="1.68" rot="MR270"/>
+<element name="R14" library="resistor" package="R0603" value="0 Ohm" x="14.78" y="6.13" rot="MR270"/>
 <element name="U$4" library="LM62" package="TO92-" value="LM62TO-92" x="28.78" y="32.4"/>
 <element name="R15" library="resistor" package="R0603" value="22" x="15.69" y="21.83" rot="R180"/>
