File: Electronics/SmartCup.sch (EAGLE design)
At the start: 51 parts, among them IC1 REG1117, IC2 REG1117, SW1 SPST_TACT-EVQQ2

Commit message: Board update
Parts:
- removed U$2: TC54VC300, TC54VC27:TC54VC300
- D1: device adafruit:DIODESMA -> adafruit:DIODE_SOD-123FL
- Q1: device adafruit:MOSFET-NREFLOW -> adafruit:MOSFET-NSOT223
Connections:
- removed net N$1: Q1.G, U$2.VOUT
- removed net N$20: C10.1, C11.1, C12.1, C13.1, C5.1, C6.1, U$1.AVCC, U$1.AVCC1, U$1.UVCC, U$1.VBUS, U$1.VCC, U$1.VCC1
- net GND: now also Q1.S; no longer Q1.D
- net LIPO_OUT: now also Q1.G; no longer U$2.VIN
- net N$8: now also Q1.D; no longer Q1.S, U$2.VSS
- net VCC: now also C10.1, C11.1, C12.1, C13.1, C5.1, C6.1, U$1.AVCC, U$1.AVCC1, U$1.UVCC, U$1.VBUS, U$1.VCC, U$1.VCC1
Other:
- moved on the sheet: Q1

Commit message: SolidWorks model
Parts:
- R10, R11, R13, R14, R4, R5, R7, R8: value 100m -> 0 Ohm
- R12, R3, R6, R9: value 100m -> 165 Ohm
Changed lines of the file:
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@@
 <grid distance="0.1" unitdist="inch" unit="inch" style="lines" multiple="1" display="no" altdistance="0.01" altunitdist="inch" altunit="inch"/>
 <layers>
-<layer number="1" name="Top" color="4" fill="1" visible="yes" active="no"/>
-<layer number="16" name="Bottom" color="1" fill="1" visible="yes" active="no"/>
-<layer number="17" name="Pads" color="2" fill="1" visible="yes" active="no"/>
-<layer number="18" name="Vias" color="2" fill="1" visible="yes" active="no"/>
-<layer number="19" name="Unrouted" color="6" fill="1" visible="yes" active="no"/>
-<layer number="20" name="Dimension" color="15" fill="1" visible="yes" active="no"/>
-<layer number="21" name="tPlace" color="7" fill="1" visible="yes" active="no"/>
-<layer number="22" name="bPlace" color="7" fill="1" visible="yes" active="no"/>
-<layer number="23" name="tOrigins" color="15" fill="1" visible="yes" active="no"/>
-<layer number="24" name="bOrigins" color="15" fill="1" visible="yes" active="no"/>
-<layer number="25" name="tNames" color="7" fill="1" visible="yes" active="no"/>
-<layer number="26" name="bNames" color="7" fill="1" visible="yes" active="no"/>
-<layer number="27" name="tValues" color="7" fill="1" visible="yes" active="no"/>
-<layer number="28" name="bValues" color="7" fill="1" visible="yes" active="no"/>
+<layer number="1" name="Top" color="4" fill="1" visible="no" active="no"/>
+<layer number="16" name="Bottom" color="1" fill="1" visible="no" active="no"/>
+<layer number="17" name="Pads" color="2" fill="1" visible="no" active="no"/>
+<layer number="18" name="Vias" color="2" fill="1" visible="no" active="no"/>
+<layer number="19" name="Unrouted" color="6" fill="1" visible="no" active="no"/>
+<layer number="20" name="Dimension" color="15" fill="1" visible="no" active="no"/>
+<layer number="21" name="tPlace" color="7" fill="1" visible="no" active="no"/>
+<layer number="22" name="bPlace" color="7" fill="1" visible="no" active="no"/>
+<layer number="23" name="tOrigins" color="15" fill="1" visible="no" active="no"/>
+<layer number="24" name="bOrigins" color="15" fill="1" visible="no" active="no"/>
+<layer number="25" name="tNames" color="7" fill="1" visible="no" active="no"/>
+<layer number="26" name="bNames" color="7" fill="1" visible="no" active="no"/>
+<layer number="27" name="tValues" color="7" fill="1" visible="no" active="no"/>
+<layer number="28" name="bValues" color="7" fill="1" visible="no" active="no"/>
 <layer number="29" name="tStop" color="7" fill="3" visible="no" active="no"/>
 <layer number="30" name="bStop" color="7" fill="6" visible="no" active="no"/>
@@
 <layer number="35" name="tGlue" color="7" fill="4" visible="no" active="no"/>
 <layer number="36" name="bGlue" color="7" fill="5" visible="no" active="no"/>
-<layer number="37" name="tTest" color="7" fill="1" visible="yes" active="no"/>
-<layer number="38" name="bTest" color="7" fill="1" visible="yes" active="no"/>
+<layer number="37" name="tTest" color="7" fill="1" visible="no" active="no"/>
+<layer number="38" name="bTest" color="7" fill="1" visible="no" active="no"/>
 <layer number="39" name="tKeepout" color="4" fill="11" visible="no" active="no"/>
 <layer number="40" name="bKeepout" color="1" fill="11" visible="no" active="no"/>
@@
 <layer number="44" name="Drills" color="7" fill="1" visible="no" active="no"/>
 <layer number="45" name="Holes" color="7" fill="1" visible="no" active="no"/>
-<layer number="46" name="Milling" color="3" fill="1" visible="yes" active="no"/>
-<layer number="47" name="Measures" color="7" fill="1" visible="yes" active="no"/>
-<layer number="48" name="Document" color="7" fill="1" visible="yes" active="no"/>
-<layer number="49" name="Reference" color="7" fill="1" visible="yes" active="no"/>
-<layer number="50" name="dxf" color="7" fill="1" visible="yes" active="no"/>
-<layer number="51" name="tDocu" color="7" fill="1" visible="yes" active="no"/>
-<layer number="52" name="bDocu" color="7" fill="1" visible="yes" active="no"/>
-<layer number="53" name="tGND_GNDA" color="7" fill="9" visible="yes" active="no"/>
-<layer number="54" name="bGND_GNDA" color="1" fill="9" visible="yes" active="no"/>
-<layer number="56" name="wert" color="7" fill="1" visible="yes" active="no"/>
-<layer number="57" name="tCAD" color="7" fill="1" visible="yes" active="no"/>
+<layer number="46" name="Milling" color="3" fill="1" visible="no" active="no"/>
+<layer number="47" name="Measures" color="7" fill="1" visible="no" active="no"/>
+<layer number="48" name="Document" color="7" fill="1" visible="no" active="no"/>
+<layer number="49" name="Reference" color="7" fill="1" visible="no" active="no"/>
+<layer number="50" name="dxf" color="7" fill="1" visible="no" active="no"/>
+<layer number="51" name="tDocu" color="7" fill="1" visible="no" active="no"/>
+<layer number="52" name="bDocu" color="7" fill="1" visible="no" active="no"/>
+<layer number="53" name="tGND_GNDA" color="7" fill="9" visible="no" active="no"/>
+<layer number="54" name="bGND_GNDA" color="1" fill="9" visible="no" active="no"/>
+<layer number="56" name="wert" color="7" fill="1" visible="no" active="no"/>
+<layer number="57" name="tCAD" color="7" fill="1" visible="no" active="no"/>
 <layer number="91" name="Nets" color="2" fill="1" visible="yes" active="yes"/>
 <layer number="92" name="Busses" color="1" fill="1" visible="yes" active="yes"/>
@@
 <part name="P+3" library="supply1" deviceset="VCC" device=""/>
 <part name="P+1" library="supply1" deviceset="VCC" device=""/>
-<part name="R3" library="resistor" deviceset="R-EU_" device="R0603" value="100m"/>
-<part name="R4" library="resistor" deviceset="R-EU_" device="R0603" value="100m"/>
-<part name="R5" library="resistor" deviceset="R-EU_" device="R0603" value="100m"/>
+<part name="R3" library="resistor" deviceset="R-EU_" device="R0603" value="165 Ohm"/>
+<part name="R4" library="resistor" deviceset="R-EU_" device="R0603" value="0 Ohm"/>
+<part name="R5" library="resistor" deviceset="R-EU_" device="R0603" value="0 Ohm"/>
 <part name="LED1" library="led" deviceset="GM1WA55311A" device=""/>
 <part name="P+4" library="supply1" deviceset="VCC" device=""/>
-<part name="R6" library="resistor" deviceset="R-EU_" device="R0603" value="100m"/>
-<part name="R7" library="resistor" deviceset="R-EU_" device="R0603" value="100m"/>
-<part name="R8" library="resistor" deviceset="R-EU_" device="R0603" value="100m"/>
+<part name="R6" library="resistor" deviceset="R-EU_" device="R0603" value="165 Ohm"/>
+<part name="R7" library="resistor" deviceset="R-EU_" device="R0603" value="0 Ohm"/>
+<part name="R8" library="resistor" deviceset="R-EU_" device="R0603" value="0 Ohm"/>
 <part name="LED2" library="led" deviceset="GM1WA55311A" device=""/>
 <part name="P+5" library="supply1" deviceset="VCC" device=""/>
-<part name="R9" library="resistor" deviceset="R-EU_" device="R0603" value="100m"/>
-<part name="R10" library="resistor" deviceset="R-EU_" device="R0603" value="100m"/>
-<part name="R11" library="resistor" deviceset="R-EU_" device="R0603" value="100m"/>
+<part name="R9" library="resistor" deviceset="R-EU_" device="R0603" value="165 Ohm"/>
+<part name="R10" library="resistor" deviceset="R-EU_" device="R0603" value="0 Ohm"/>
+<part name="R11" library="resistor" deviceset="R-EU_" device="R0603" value="0 Ohm"/>
 <part name="GND15" library="supply1" deviceset="GND" device=""/>
 <part name="C10" library="resistor" deviceset="C-EU" device="C0603" value="100nF"/>
@@
 <part name="LED3" library="led" deviceset="GM1WA55311A" device=""/>
 <part name="P+6" library="supply1" deviceset="VCC" device=""/>
-<part name="R12" library="resistor" deviceset="R-EU_" device="R0603" value="100m"/>
-<part name="R13" library="resistor" deviceset="R-EU_" device="R0603" value="100m"/>
-<part name="R14" library="resistor" deviceset="R-EU_" device="R0603" value="100m"/>
+<part name="R12" library="resistor" deviceset="R-EU_" device="R0603" value="165 Ohm"/>
+<part name="R13" library="resistor" deviceset="R-EU_" device="R0603" value="0 Ohm"/>
+<part name="R14" library="resistor" deviceset="R-EU_" device="R0603" value="0 Ohm"/>
 <part name="U$4" library="LM62" deviceset="LM62" device="TO-92" value="LM62TO-92"/>
 <part name="GND19" library="supply1" deviceset="GND" device=""/>
@@
 <part name="R15" library="resistor" deviceset="R-EU_" device="R0603" value="22"/>
 <part name="R16" library="resistor" deviceset="R-EU_" device="R0603" value="22"/>
-<part name="GND25" library="supply1" deviceset="GND" device=""/>
 <part name="U$6" library="BOURNS" deviceset="BOURNS_PWR" device=""/>
 <part name="U$7" library="BOURNS" deviceset="BOURNS_PWR" device=""/>
@@
 <instance part="R15" gate="G$1" x="30.48" y="154.94" rot="MR90"/>
 <instance part="R16" gate="G$1" x="38.1" y="154.94" rot="R270"/>
-<instance part="GND25" gate="1" x="251.46" y="30.48"/>
 <instance part="U$6" gate="G$1" x="185.42" y="76.2" rot="R180"/>
 <instance part="U$7" gate="G$1" x="185.42" y="91.44" rot="R180"/>
